File: canhub/canhub.kicad_sch (KiCad schematic)
At the start: 12 parts

Commit message: Update schematic
Parts:
- removed J? (x2): Conn_01x05_Female, symbol Connector:Conn_01x05_Female
- added J5: Master1, symbol Connector:Conn_01x05_Female
- added J6: Master2, symbol Connector:Conn_01x05_Female
- added T1: 6_POL_TOGGLE_SWITCH, symbol New_Library:6_POL_TOGGLE_SWITCH
- J1: renamed from J?; value Conn_01x05_Male -> In
- J10: renamed from J?; value Conn_01x05_Female -> Slave7
- J11: renamed from J?; value Conn_01x05_Female -> Slave8
- J12: renamed from J?; value Conn_01x05_Female -> Out
- J2: renamed from J?; value Conn_01x05_Female -> Slave1
- J3: renamed from J?; value Conn_01x05_Female -> Slave2
- J4: renamed from J?; value Conn_01x05_Female -> Slave3
- J7: renamed from J?; value Conn_01x05_Female -> Slave4
- J8: renamed from J?; value Conn_01x05_Female -> Slave5
- J9: renamed from J?; value Conn_01x05_Female -> Slave6
Connections:
- net at J1.1 (Pin_1), J10.1 (Pin_1), J11.1 (Pin_1)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: now also J5.1 (Pin_1), J6.1 (Pin_1)
- net at J1.2 (Pin_2), J10.2 (Pin_2), J11.2 (Pin_2)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: now also J5.2 (Pin_2), J6.2 (Pin_2)
- net at J1.3 (Pin_3), J10.3 (Pin_3), J11.3 (Pin_3)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: now also J5.3 (Pin_3), J6.3 (Pin_3)
- net at J1.4 (Pin_4), J10.4 (Pin_4), J11.4 (Pin_4)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: now also T1.1
- net at J1.5 (Pin_5), J10.5 (Pin_5), J11.5 (Pin_5)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: now also T1.2
- new net: J5.4 (Pin_4), T1.3
- new net: J5.5 (Pin_5), T1.5
- new net: J6.4 (Pin_4), T1.4
- new net: J6.5 (Pin_5), T1.6
